Commit message: 瞎调了一些参数

File: resources/robots/pointfoot/PF_P441B/urdf/robot.urdf (robot description, URDF)
Before this commit: robot point_foot, 12 links, 11 joints
Links:
- link abad_L_Link: mass 1.59 -> 1.614
- link abad_R_Link: mass 1.59 -> 1.614
- link base_Link: mass 8.49 -> 8.557; geometry collision box size=0.37 0.26 0.14; visual mesh filename=../meshes/base_Link.STL
- link foot_L_Link: mass 0.16 -> 0.157; geometry collision sphere radius=0.03; visual mesh filename=../meshes/foot_L_Link.STL
- link foot_R_Link: mass 0.16 -> 0.157; geometry collision sphere radius=0.03; visual mesh filename=../meshes/foot_R_Link.STL
- link hip_L_Link: mass 2.39 -> 2.435; geometry collision cylinder length=0.15 radius=0.035; visual mesh filename=../meshes/hip_L_Link.STL
- link hip_R_Link: mass 2.39 -> 2.435; geometry collision cylinder length=0.15 radius=0.035; visual mesh filename=../meshes/hip_R_Link.STL
- link knee_L_Link: mass 0.38 -> 0.573
- link knee_R_Link: mass 0.38 -> 0.573
Joints:
- joint abad_L_Joint: limit lower=-0.38397 upper=1.39626 effort=80.0 velocity=15.0 -> lower=-0.38397 upper=1.39626 effort=80.0 velocity=20.0; origin xyz=16.2E-03 105E-03 -90.76E-03 rpy=0 0 0 -> xyz=0.01241 0.10494 -0.09876 rpy=0 0 0
- joint abad_R_Joint: limit lower=-1.39626 upper=0.38397 effort=80.0 velocity=15.0 -> lower=-1.39626 upper=0.38397 effort=80.0 velocity=20.0; origin xyz=16.2E-03 -105E-03 -90.76E-03 rpy=0 0 0 -> xyz=0.01241 -0.10494 -0.09876 rpy=0 0 0
- joint contact_L_Joint: origin xyz=0 0 -0.032 rpy=0 0 0 -> xyz=0 0 -0.03 rpy=0 0 0
- joint contact_R_Joint: origin xyz=0 0 -0.032 rpy=0 0 0 -> xyz=0 0 -0.03 rpy=0 0 0
- joint foot_L_Joint: origin xyz=0.150 0 -0.2598 rpy=0 0 0 -> xyz=0.15 0 -0.25981 rpy=0 0 0
- joint foot_R_Joint: origin xyz=0.150 0 -0.2598 rpy=0 0 0 -> xyz=0.15 0 -0.25981 rpy=0 0 0
- joint hip_L_Joint: limit lower=-1.012291 upper=1.396263 effort=80.0 velocity=15.0 -> lower=-1.012291 upper=1.518436 effort=80.0 velocity=20.0; origin xyz=-77E-03 20.5E-03 0 rpy=0 0 0 -> xyz=-0.07696 0.02066 0 rpy=0 0 0
- joint hip_R_Joint: limit lower=-1.396263 upper=1.012291 effort=80.0 velocity=15.0 -> lower=-1.518436 upper=1.012291 effort=80.0 velocity=20.0; origin xyz=-77E-03 -20.5E-03 0 rpy=0 0 0 -> xyz=-0.07696 -0.02066 0 rpy=0 0 0
- joint knee_L_Joint: limit lower=-0.872665 upper=1.361357 effort=80 velocity=15 -> lower=-0.872665 upper=1.396263 effort=80 velocity=20; origin xyz=-150E-03 -20.5E-03 -0.25981 rpy=0 0 0 -> xyz=-0.15004 -0.02018 -0.25981 rpy=0 0 0
- joint knee_R_Joint: limit lower=-1.361357 upper=0.872665 effort=80 velocity=15 -> lower=-1.396263 upper=0.872665 effort=80 velocity=50; origin xyz=-150E-03 20.5E-03 -0.25981 rpy=0 0 0 -> xyz=-0.15004 0.02018 -0.25981 rpy=0 0 0

File: resources/robots/pointfoot/PF_P441C/urdf/robot.urdf (robot description, URDF)
Before this commit: robot point_foot, 12 links, 11 joints
Links:
- link abad_L_Link: mass 1.560 -> 1.614
- link abad_R_Link: mass 1.560 -> 1.614
- link base_Link: mass 9.567 -> 8.557; geometry collision box size=0.37 0.26 0.14; visual mesh filename=../meshes/base_Link.STL
- link foot_L_Link: mass 0.197 -> 0.157; geometry collision sphere radius=0.03; visual mesh filename=../meshes/foot_L_Link.STL
- link foot_R_Link: mass 0.176 -> 0.157; geometry collision sphere radius=0.03; visual mesh filename=../meshes/foot_R_Link.STL
- link hip_L_Link: mass 2.388 -> 2.435; geometry collision cylinder length=0.15 radius=0.035; visual mesh filename=../meshes/hip_L_Link.STL
- link hip_R_Link: mass 2.388 -> 2.435; geometry collision cylinder length=0.15 radius=0.035; visual mesh filename=../meshes/hip_R_Link.STL
- link knee_L_Link: mass 0.496 -> 0.573
- link knee_R_Link: mass 0.496 -> 0.573
Joints:
- joint abad_L_Joint: limit lower=-0.38397 upper=1.39626 effort=80.0 velocity=15.0 -> lower=-0.38397 upper=1.39626 effort=80.0 velocity=20.0; origin xyz=0.039 0.1095 -0.08725 rpy=0 0 0 -> xyz=0.01241 0.10494 -0.09876 rpy=0 0 0
- joint abad_R_Joint: limit lower=-1.39626 upper=0.38397 effort=80.0 velocity=15.0 -> lower=-1.39626 upper=0.38397 effort=80.0 velocity=20.0; origin xyz=0.039 -0.1095 -0.08725 rpy=0 0 0 -> xyz=0.01241 -0.10494 -0.09876 rpy=0 0 0
- joint contact_L_Joint: origin xyz=0 0 -0.032 rpy=0 0 0 -> xyz=0 0 -0.03 rpy=0 0 0
- joint contact_R_Joint: origin xyz=0 0 -0.032 rpy=0 0 0 -> xyz=0 0 -0.03 rpy=0 0 0
- joint foot_L_Joint: origin xyz=0.150 0 -0.25981 rpy=0 0 0 -> xyz=0.15 0 -0.25981 rpy=0 0 0
- joint foot_R_Joint: origin xyz=0.150 0 -0.25981 rpy=0 0 0 -> xyz=0.15 0 -0.25981 rpy=0 0 0
- joint hip_L_Joint: limit lower=-1.012291 upper=1.396263 effort=80.0 velocity=15.0 -> lower=-1.012291 upper=1.518436 effort=80.0 velocity=20.0; origin xyz=-0.077 0.02050 0 rpy=0 0 0 -> xyz=-0.07696 0.02066 0 rpy=0 0 0
- joint hip_R_Joint: limit lower=-1.396263 upper=1.012291 effort=80.0 velocity=15.0 -> lower=-1.518436 upper=1.012291 effort=80.0 velocity=20.0; origin xyz=-0.077 -0.02050 0 rpy=0 0 0 -> xyz=-0.07696 -0.02066 0 rpy=0 0 0
- joint knee_L_Joint: limit lower=-0.872665 upper=1.361357 effort=80 velocity=15 -> lower=-0.872665 upper=1.396263 effort=80 velocity=20; origin xyz=-0.1500 -0.02050 -0.25981 rpy=0 0 0 -> xyz=-0.15004 -0.02018 -0.25981 rpy=0 0 0
- joint knee_R_Joint: limit lower=-1.361357 upper=0.872665 effort=80 velocity=15 -> lower=-1.396263 upper=0.872665 effort=80 velocity=50; origin xyz=-0.1500 0.02050 -0.25981 rpy=0 0 0 -> xyz=-0.15004 0.02018 -0.25981 rpy=0 0 0

File: resources/robots/pointfoot/PF_P441C2/urdf/robot.urdf (robot description, URDF)
Before this commit: robot point_foot, 12 links, 11 joints
Links:
- link abad_L_Link: mass 1.48 -> 1.614
- link abad_R_Link: mass 1.560 -> 1.614
- link base_Link: mass 9.417 -> 8.557; geometry collision box size=0.37 0.26 0.14; visual mesh filename=../meshes/base_Link.STL
- link foot_L_Link: mass 0.188 -> 0.157; geometry collision sphere radius=0.03; visual mesh filename=../meshes/foot_L_Link.STL
- link foot_R_Link: mass 0.188 -> 0.157; geometry collision sphere radius=0.03; visual mesh filename=../meshes/foot_R_Link.STL
- link hip_L_Link: mass 2.257 -> 2.435; geometry collision cylinder length=0.15 radius=0.035; visual mesh filename=../meshes/hip_L_Link.STL
- link hip_R_Link: mass 2.257 -> 2.435; geometry collision cylinder length=0.15 radius=0.035; visual mesh filename=../meshes/hip_R_Link.STL
- link knee_L_Link: mass 0.542 -> 0.573
- link knee_R_Link: mass 0.496 -> 0.573
Joints:
- joint abad_L_Joint: limit lower=-0.38397 upper=1.39626 effort=80.0 velocity=15.0 -> lower=-0.38397 upper=1.39626 effort=80.0 velocity=20.0; origin xyz=23.76E-03 105E-03 -93.8E-03 rpy=0 0 0 -> xyz=0.01241 0.10494 -0.09876 rpy=0 0 0
- joint abad_R_Joint: limit lower=-1.39626 upper=0.38397 effort=80.0 velocity=15.0 -> lower=-1.39626 upper=0.38397 effort=80.0 velocity=20.0; origin xyz=23.76E-03 -105E-03 -93.8E-03 rpy=0 0 0 -> xyz=0.01241 -0.10494 -0.09876 rpy=0 0 0
- joint contact_L_Joint: origin xyz=0 0 -0.032 rpy=0 0 0 -> xyz=0 0 -0.03 rpy=0 0 0
- joint contact_R_Joint: origin xyz=0 0 -0.032 rpy=0 0 0 -> xyz=0 0 -0.03 rpy=0 0 0
- joint foot_L_Joint: origin xyz=0.150 0 -0.25981 rpy=0 0 0 -> xyz=0.15 0 -0.25981 rpy=0 0 0
- joint foot_R_Joint: origin xyz=0.150 0 -0.25981 rpy=0 0 0 -> xyz=0.15 0 -0.25981 rpy=0 0 0
- joint hip_L_Joint: limit lower=-1.012291 upper=1.396263 effort=80.0 velocity=15.0 -> lower=-1.012291 upper=1.518436 effort=80.0 velocity=20.0; origin xyz=-0.077 0.02050 0 rpy=0 0 0 -> xyz=-0.07696 0.02066 0 rpy=0 0 0
- joint hip_R_Joint: limit lower=-1.396263 upper=1.012291 effort=80.0 velocity=15.0 -> lower=-1.518436 upper=1.012291 effort=80.0 velocity=20.0; origin xyz=-0.077 -0.02050 0 rpy=0 0 0 -> xyz=-0.07696 -0.02066 0 rpy=0 0 0
- joint knee_L_Joint: limit lower=-0.872665 upper=1.361357 effort=80 velocity=15 -> lower=-0.872665 upper=1.396263 effort=80 velocity=20; origin xyz=-0.1500 -0.02050 -0.25981 rpy=0 0 0 -> xyz=-0.15004 -0.02018 -0.25981 rpy=0 0 0
- joint knee_R_Joint: limit lower=-1.361357 upper=0.872665 effort=80 velocity=15 -> lower=-1.396263 upper=0.872665 effort=80 velocity=50; origin xyz=-0.1500 0.02050 -0.25981 rpy=0 0 0 -> xyz=-0.15004 0.02018 -0.25981 rpy=0 0 0
